File: Peak-Detector/Peak-Detector.kicad_sch (KiCad schematic)
At the start: 20 parts, among them U1 LMH6658, U2 LMH6658

Commit message: adding Nuclear-Phoenix-inspired peak detector schematic
Parts:
- added C11, C16: 0.1uF, Capacitor_SMD:C_0603_1608Metric, symbol device:C
- added C12, C13, C17, C18: 10nF, Capacitor_SMD:C_0603_1608Metric, symbol device:C
- added C14, C19: 10n, Capacitor_SMD:C_0603_1608Metric, symbol device:C
- added C15: 470pF, Capacitor_SMD:C_0603_1608Metric, symbol device:C
- added D5, D6: D_Schottky, Diode_SMD:D_SOD-523, symbol My_Symbol_Library:D_Schottky
- added Q1: 2N7002, Package_TO_SOT_SMD:SOT-23, symbol Transistor_FET:2N7002
- added R5, R7: 100, Capacitor_SMD:C_0603_1608Metric, symbol device:R
- added R6: 1k, Capacitor_SMD:C_0603_1608Metric, symbol device:R
- added U3, U4: OPA357AIDBVR, symbol Simulation_SPICE:OPAMP
Connections:
- net AMP1: now also U3.1 (+)
- net GNDA: now also C11.1, C12.1, C13.2, C14.2, C15.1, C16.1, C17.1, C18.2, C19.2, Q1.2 (S)
- net VCC: now also C13.1, C14.1, C18.1, C19.1, U3.4 (V+), U4.4 (V+)
- net VEE: now also C11.2, C12.2, C15.2, C16.2, C17.2, R5.1, R6.2, U3.2 (-), U3.5 (V-), U4.1 (+), U4.5 (V-)
- new net: D6.1 (K), R5.2
- new net: D5.1 (K), D6.2 (A), R7.2
- new net: Q1.3 (D), R6.1
- new net: D5.2 (A), U3.3
- new net PEAK: R7.1, U4.2 (-), U4.3
- new net RST: Q1.1 (G)
