File: Peak-Detector/Peak-Detector.kicad_sch (KiCad schematic)
At the start: 37 parts, among them Q1 2N7002, U1 LMH6658, U2 LMH6658, U3 OPA357AIDBVR, U4 OPA357AIDBVR

Commit message: adding peak detector and comparator
Connections:
- net VEE: no longer C15.2, R5.1, R6.2, U3.2 (-), U4.1 (+)
- new net: C15.2, R5.1, R6.2, U3.2 (-), U4.1 (+)
Changed lines of the file:
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@@
   (junction (at 237.49 76.2) (diameter 0) (color 0 0 0 0)
   )
-  (junction (at 179.07 59.69) (diameter 0) (color 0 0 0 0)
-  )
   (junction (at 59.69 125.73) (diameter 0) (color 0 0 0 0)
   )
@@
     (stroke (width 0) (type default))
   )
-  (wire (pts (xy 179.07 59.69) (xy 218.44 59.69))
-    (stroke (width 0) (type default))
-  )
   (wire (pts (xy 91.44 139.7) (xy 77.47 139.7))
     (stroke (width 0) (type default))
   )
-  (wire (pts (xy 171.45 59.69) (xy 179.07 59.69))
-    (stroke (width 0) (type default))
-  )
+  (wire (pts (xy 171.45 59.69) (xy 218.44 59.69))
+    (stroke (width 0) (type default))
+  )

Commit message: adding old peak detetion schematic
Parts:
- added C20: 10pF, Capacitor_SMD:C_0603_1608Metric, symbol device:C
- added C21: 10uF, Capacitor_SMD:C_0603_1608Metric, symbol device:C
- added C22: 20nF, Capacitor_SMD:C_0603_1608Metric, symbol device:C
- added C23: 0.1uF, Capacitor_SMD:C_0603_1608Metric, symbol device:C
- added D7, D8: Schottky, Diode_SMD:D_SOD-523, symbol My_Symbol_Library:D_Schottky
- added R10, R9: 100k, Capacitor_SMD:C_0603_1608Metric, symbol device:R
- added R11: 249, Capacitor_SMD:C_0603_1608Metric, symbol device:R
- added R12: 10k, Capacitor_SMD:C_0603_1608Metric, symbol device:R
- added U5, U6: LT1807, symbol Simulation_SPICE:OPAMP
Connections:
- net GNDA: now also C21.2, C22.1, C23.2, R11.2, R9.2, U5.5 (V-), U6.5 (V-)
- net VCC: now also C21.1, C23.1, U5.4 (V+), U6.4 (V+)
- net VEE: now also C15.2, R5.1, R6.2, U3.2 (-), U4.1 (+)
- new net: D7.2 (A), D8.1 (K), U6.3
- new net: D8.2 (A), R10.1, R9.1, U6.2 (-)
- new net: C20.2, R11.1, R12.1, U5.2 (-)
- new net Amp: C20.1, R12.2, U5.3, U6.1 (+)
- new net Peak: C22.2, D7.1 (K), R10.2
- new net SiPM: U5.1 (+)
Other:
- moved on the sheet: C10, C6, C7, C8, C9, D3, D4, R3, R4, U2

Commit message: optimizing some components
Parts:
- added C24, C27, C29, C32: 0.1uF, Capacitor_SMD:C_0603_1608Metric, symbol device:C
- added C25, C26, C30, C31: 10nF, Capacitor_SMD:C_0603_1608Metric, symbol device:C
- added C28: 2nF, Capacitor_SMD:C_0603_1608Metric, symbol device:C
- added D10, D9: D_Schottky, Diode_SMD:D_SOD-523, symbol My_Symbol_Library:D_Schottky
- added P1: CONN_01X04, MyFootprints:PinHeader4_bigger_SiPM, symbol conn:CONN_01X04
- added Q2: 2N7002, Package_TO_SOT_SMD:SOT-23, symbol Transistor_FET:2N7002
- added R13: 49.9, Capacitor_SMD:C_0603_1608Metric, symbol device:R
- added R14: 1k, Capacitor_SMD:C_0603_1608Metric, symbol device:R
- added R15, R18, R20: 10k, Capacitor_SMD:C_0603_1608Metric, symbol device:R
- added R17, R21: 100, Capacitor_SMD:C_0603_1608Metric, symbol device:R
- added R19: 10, Capacitor_SMD:C_0603_1608Metric, symbol device:R
- added R8: 47k, Capacitor_SMD:C_0603_1608Metric, symbol device:R
- added U7, U8: LMH6658, Package_SO:SOIC-8_3.9x4.9mm_P1.27mm, symbol My_Library:LMH6658
Connections:
- net AMP1: now also R15.1, U7.1 (OUTA), U7.5 (+INB), U8.5 (+INB)
- net GNDA: now also C24.1, C25.1, C26.2, C27.2, C28.1, C29.1, C30.1, C31.2, C32.2, P1.3 (P3), Q2.2 (S), R14.2, R18.1, R21.1, R8.2
- net SiPM: now also P1.4 (P4), R13.1, R8.1
- net VCC: now also C26.1, C27.1, C31.1, C32.1, R20.1, U7.8 (V+), U8.8 (V+)
- net VEE: now also C24.2, C25.2, C29.2, C30.2, U7.4 (V-), U8.4 (V-)
- new net: C28.2, D10.1 (K), R18.2, R19.2, U8.3 (+INA)
- new net: D10.2 (A), D9.2 (A), R17.2, U7.7 (OUTB)
- new net: Q2.3 (D), R19.1
- new net: R20.2, R21.2, U8.6 (-INB)
- new net: D9.1 (K), U7.6 (-INB)
- new net: R14.1, R15.2, U7.2 (-INA)
- new net: R13.2, U7.3 (+INA)
- new net FAST: P1.1 (P1)
- new net HV: P1.2 (P2)
- new net SNG1: R17.1, U8.1 (OUTA), U8.2 (-INA)
- new net TRG: U8.7 (OUTB)
- new net TriggerReset1: Q2.1 (G)
Other:
- note added: "Good"
- moved on the sheet: C1, C10, C2, C3, C4, C5, C6, C7, C8, C9, D1, D2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
