File: CosmicWatch_detector_v30/CosmicWatch.kicad_sch (KiCad schematic)
At the start: 86 parts, among them J3 RJ45, P1 CONN_01X04, P10 CONN_02X02, P11 CONN_01X01, P12 CONN_01X01, P13 CONN_01X01, P14 CONN_01X01, P15 CONN_02X04, P16 CONN_01X02, P19 CONN_01X01, P2 CONN_01X01, P3 CONN_01X04, P4 CONN_01X04, P5 CONN_01X02, P7 CONN_01X01, P8 CONN_01X01, Q2 2N7002, SW1 RESET, U1 MAX5026, U13 TS5A1066, U16 UMCC, U17 UMCC, U2 SiPM_MicroFJ−300XX−TSV, U22 UMCC, U23 UMCC, U3 MMCX, U4 TS5A1066, U5 LMH6658, U5 RasberryPi_Pico, U6 LMH6658, U7 TPS6040X, U8 sd_card_socket

Commit message: moved MOSFET
Parts:
- C24: value 10nF -> 2nF
- R14: value 1k -> 10k
Connections:
- net GNDA: now also R14.1
- net SiPM: now also R9.1
- net TriggerReset1: now also Q2.1 (G)
- net at C24.2, R12.1, R14.2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: now also Q2.3 (D)
Other:
- moved on the sheet: P4, Q2
Changed lines of the file:
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@@
   (junction (at 115.57 210.82) (diameter 0) (color 0 0 0 0)
   )
+  (junction (at 140.716 125.73) (diameter 0) (color 0 0 0 0)
+  )
   (junction (at 110.49 228.6) (diameter 0) (color 0 0 0 0)
   )
@@
     (stroke (width 0) (type default))
   )
-  (wire (pts (xy 134.62 125.73) (xy 165.1 125.73))
+  (wire (pts (xy 134.62 125.73) (xy 140.716 125.73))
     (stroke (width 0) (type default))
   )
@@
     (stroke (width 0) (type default))
   )
-  (wire (pts (xy 44.45 125.73) (xy 45.085 125.73))
+  (wire (pts (xy 44.45 125.73) (xy 45.72 125.73))
     (stroke (width 0) (type default))
   )
@@
     (stroke (width 0) (type default))
   )
+  (wire (pts (xy 140.716 125.73) (xy 140.716 141.732))
+    (stroke (width 0) (type default))
+  )
   (wire (pts (xy 63.5 55.88) (xy 68.072 55.88))
     (stroke (width 0) (type default))
@@
     (stroke (width 0) (type default))
   )
+  (wire (pts (xy 140.716 125.73) (xy 165.1 125.73))
+    (stroke (width 0) (type default))
+  )
   (wire (pts (xy 194.31 111.76) (xy 196.85 111.76))
     (stroke (width 0) (type default))
@@
     )
   )
-  (global_label "3.3V" (shape input) (at 389.89 177.8 180) (fields_autoplaced)
+  (global_label "3.3V" (shape input) (at 360.934 153.67 180) (fields_autoplaced)
     (effects (font (size 1.524 1.524)) (justify right))
-    (property "Intersheetrefs" "${INTERSHEET_REFS}" (at 6.35 50.8 0)
+    (property "Intersheetrefs" "${INTERSHEET_REFS}" (at -22.606 26.67 0)
       (effects (font (size 1.27 1.27)) hide)
     )
@@
     )
   )
+  (global_label "TriggerReset1" (shape input) (at 133.096 146.812 180) (fields_autoplaced)
+    (effects (font (size 1.524 1.524)) (justify right))
+    (property "Intersheetrefs" "${INTERSHEET_REFS}" (at 114.8643 146.812 0)
+      (effects (font (size 1.27 1.27)) (justify right) hide)
+    )
+  )
   (global_label "VEE" (shape input) (at 368.427 111.379 180) (fields_autoplaced)
     (effects (font (size 1.524 1.524)) (justify right))
@@
     )
   )
-  (global_label "SDA" (shape input) (at 389.89 185.42 180) (fields_autoplaced)
+  (global_label "SDA" (shape input) (at 360.934 161.29 180) (fields_autoplaced)
     (effects (font (size 1.524 1.524)) (justify right))
-    (property "Intersheetrefs" "${INTERSHEET_REFS}" (at 382.9069 185.42 0)
+    (property "Intersheetrefs" "${INTERSHEET_REFS}" (at 353.9509 161.29 0)
       (effects (font (size 1.27 1.27)) (justify right) hide)
     )
@@
     )
   )
-  (global_label "SCL" (shape input) (at 389.89 182.88 180) (fields_autoplaced)
+  (global_label "SCL" (shape input) (at 360.934 158.75 180) (fields_autoplaced)
     (effects (font (size 1.524 1.524)) (justify right))
-    (property "Intersheetrefs" "${INTERSHEET_REFS}" (at 382.9795 182.88 0)
+    (property "Intersheetrefs" "${INTERSHEET_REFS}" (at 354.0235 158.75 0)
       (effects (font (size 1.27 1.27)) (justify right) hide)
     )
@@
     )
   )
-  (symbol (lib_id "power:GNDD") (at 389.89 180.34 270) (unit 1)
+  (symbol (lib_id "power:GNDD") (at 360.934 156.21 270) (unit 1)
     (in_bom yes) (on_board yes) (dnp no)
-    (property "Reference" "#PWR0165" (at 383.54 180.34 0)
+    (property "Reference" "#PWR0165" (at 354.584 156.21 0)
       (effects (font (size 1.27 1.27)) hide)
     )
-    (property "Value" "GNDD" (at 386.6388 180.467 90)
+    (property "Value" "GNDD" (at 357.6828 156.337 90)
       (effects (font (size 1.27 1.27)) (justify right))
     )
-    (property "Footprint" "" (at 389.89 180.34 0)
+    (property "Footprint" "" (at 360.934 156.21 0)
       (effects (font (size 1.27 1.27)))
     )
-    (property "Datasheet" "" (at 389.89 180.34 0)
+    (property "Datasheet" "" (at 360.934 156.21 0)
       (effects (font (size 1.27 1.27)))
     )
@@
     )
   )
-  (symbol (lib_id "conn:CONN_01X04") (at 394.97 181.61 0) (unit 1)
+  (symbol (lib_id "conn:CONN_01X04") (at 366.014 157.48 0) (unit 1)
     (in_bom yes) (on_board yes) (dnp no)
-    (property "Reference" "P4" (at 396.9512 180.5686 0)
+    (property "Reference" "P4" (at 367.9952 156.4386 0)
       (effects (font (size 1.27 1.27)) (justify left))
     )
-    (property "Value" "CONN_01X04" (at 396.9512 182.88 0)
+    (property "Value" "CONN_01X04" (at 367.9952 158.75 0)
       (effects (font (size 1.27 1.27)) (justify left))
     )
-    (property "Footprint" "Connector_PinHeader_2.54mm:PinHeader_1x04_P2.54mm_Vertical" (at 394.97 181.61 0)
+    (property "Footprint" "Connector_PinHeader_2.54mm:PinHeader_1x04_P2.54mm_Vertical" (at 366.014 157.48 0)
       (effects (font (size 1.27 1.27)) hide)
     )
-    (property "Datasheet" "" (at 394.97 181.61 0)
+    (property "Datasheet" "" (at 366.014 157.48 0)
       (effects (font (size 1.27 1.27)))
     )
@@
       (effects (font (size 1.27 1.27)) (justify left))
     )
-    (property "Value" "10nF" (at 127.635 127 0)
+    (property "Value" "2nF" (at 127.635 127 0)
       (effects (font (size 1.27 1.27)) (justify left))
     )
@@
     )
   )
+  (symbol (lib_id "power:GNDA") (at 134.62 139.7 0) (unit 1)
+    (in_bom yes) (on_board yes) (dnp no)
+    (property "Reference" "#PWR024" (at 134.62 146.05 0)
+      (effects (font (size 1.27 1.27)) hide)
+    )
+    (property "Value" "GNDA" (at 134.747 142.9512 90)
+      (effects (font (size 1.27 1.27)) (justify right))
+    )
+    (property "Footprint" "" (at 134.62 139.7 0)
+      (effects (font (size 1.27 1.27)))
+    )
+    (property "Datasheet" "" (at 134.62 139.7 0)
+      (effects (font (size 1.27 1.27)))
+    )
+    (pin "1")
+    (instances
+      (project "Peak-Detector"
+        (path "/1a5a94c0-4994-4302-8f30-e2771c050d24"
+          (reference "#PWR024") (unit 1)
+        )
+      )
+      (project "CosmicWatch"
+        (path "/4ba73f5d-b469-4168-abd4-8f6ff03fbc45"
+          (reference "#PWR028") (unit 1)
+        )
+      )
+      (project "DC-DC-booster"
+        (path "/ee3fefaa-818f-4207-9a53-d175ff74ab66"
+          (reference "#PWR08") (unit 1)
+        )
+      )
+    )
+  )
   (symbol (lib_id "power:GNDA") (at 230.505 182.88 0) (unit 1)
     (in_bom yes) (on_board yes) (dnp no)
@@
     )
   )
-  (symbol (lib_id "Transistor_FET:2N7002") (at 132.08 144.78 0) (unit 1)
+  (symbol (lib_id "Transistor_FET:2N7002") (at 138.176 146.812 0) (unit 1)
     (in_bom yes) (on_board yes) (dnp no)
-    (property "Reference" "Q2" (at 135.89 140.97 0)
+    (property "Reference" "Q2" (at 141.986 143.002 0)
       (effects (font (size 1.27 1.27)) (justify left))
     )
-    (property "Value" "2N7002" (at 135.89 148.59 0)
+    (property "Value" "2N7002" (at 141.986 150.622 0)
       (effects (font (size 1.27 1.27)) (justify left))
     )
-    (property "Footprint" "Package_TO_SOT_SMD:SOT-23" (at 137.16 146.685 0)
+    (property "Footprint" "Package_TO_SOT_SMD:SOT-23" (at 143.256 148.717 0)
       (effects (font (size 1.27 1.27) italic) (justify left) hide)
     )
-    (property "Datasheet" "https://www.onsemi.com/pub/Collateral/NDS7002A-D.PDF" (at 132.08 144.78 0)
+    (property "Datasheet" "https://www.onsemi.com/pub/Collateral/NDS7002A-D.PDF" (at 138.176 146.812 0)
       (effects (font (size 1.27 1.27)) (justify left) hide)
     )
@@
     )
   )
-  (symbol (lib_id "power:GNDA") (at 134.62 149.86 0) (unit 1)
+  (symbol (lib_id "power:GNDA") (at 140.716 151.892 0) (unit 1)
     (in_bom yes) (on_board yes) (dnp no)
-    (property "Reference" "#PWR024" (at 134.62 156.21 0)
+    (property "Reference" "#PWR024" (at 140.716 158.242 0)
       (effects (font (size 1.27 1.27)) hide)
     )
-    (property "Value" "GNDA" (at 134.747 153.1112 90)
+    (property "Value" "GNDA" (at 140.843 155.1432 90)
       (effects (font (size 1.27 1.27)) (justify right))
     )
-    (property "Footprint" "" (at 134.62 149.86 0)
+    (property "Footprint" "" (at 140.716 151.892 0)
       (effects (font (size 1.27 1.27)))
     )
-    (property "Datasheet" "" (at 134.62 149.86 0)
+    (property "Datasheet" "" (at 140.716 151.892 0)
       (effects (font (size 1.27 1.27)))
     )
@@
       (effects (font (size 1.27 1.27)))
     )
-    (property "Value" "1k" (at 134.62 129.54 90)
+    (property "Value" "10k" (at 134.62 129.54 90)
       (effects (font (size 1.27 1.27)))
     )
