File: CosmicWatch_detector_v30/CosmicWatch.kicad_sch (KiCad schematic)
At the start: 79 parts, among them J3 RJ45, P1 CONN_01X04, P10 CONN_02X02, P11 CONN_01X01, P12 CONN_01X01, P13 CONN_01X01, P14 CONN_01X01, P15 CONN_02X04, P16 CONN_01X02, P19 CONN_01X01, P2 CONN_01X01, P3 CONN_01X04, P4 CONN_01X04, P5 CONN_01X02, P7 CONN_01X01, P8 CONN_01X01, Q2 2N7002, SW1 RESET, U1 MAX5026, U16 UMCC, U17 UMCC, U2 SiPM_MicroFJ−300XX−TSV, U3 MMCX, U5 LMH6658, U5 RasberryPi_Pico, U6 LMH6658, U7 TPS6040X, U8 sd_card_socket

Commit message: adding old peak detetion schematic
Other:
- moved on the sheet: C7
Changed lines of the file:
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@@
   (junction (at 95.25 215.9) (diameter 0) (color 0 0 0 0)
   )
-  (junction (at 68.072 55.88) (diameter 0) (color 0 0 0 0)
-  )
   (junction (at 96.52 34.29) (diameter 0) (color 0 0 0 0)
   )
@@
   (junction (at 143.51 130.81) (diameter 0) (color 0 0 0 0)
   )
+  (junction (at 74.93 55.88) (diameter 0) (color 0 0 0 0)
+  )
   (junction (at 118.11 119.38) (diameter 0) (color 0 0 0 0)
   )
@@
     (stroke (width 0) (type default))
   )
+  (wire (pts (xy 63.5 55.88) (xy 74.93 55.88))
+    (stroke (width 0) (type default))
+  )
   (wire (pts (xy 68.58 39.37) (xy 63.5 39.37))
     (stroke (width 0) (type default))
@@
     (stroke (width 0) (type default))
   )
+  (wire (pts (xy 74.93 55.88) (xy 81.28 55.88))
+    (stroke (width 0) (type default))
+  )
   (wire (pts (xy 208.28 135.89) (xy 209.55 135.89))
     (stroke (width 0) (type default))
@@
     (stroke (width 0) (type default))
   )
-  (wire (pts (xy 68.072 55.88) (xy 81.28 55.88))
-    (stroke (width 0) (type default))
-  )
   (wire (pts (xy 198.12 130.81) (xy 200.66 130.81))
     (stroke (width 0) (type default))
   )
-  (wire (pts (xy 63.5 55.88) (xy 68.072 55.88))
-    (stroke (width 0) (type default))
-  )
   (wire (pts (xy 367.03 25.4) (xy 368.554 25.4))
     (stroke (width 0) (type default))
@@
     )
   )
-  (symbol (lib_id "power:GNDA") (at 68.072 63.5 0) (unit 1)
+  (symbol (lib_id "power:GNDA") (at 74.93 63.5 0) (unit 1)
     (in_bom yes) (on_board yes) (dnp no)
-    (property "Reference" "#PWR015" (at 68.072 69.85 0)
+    (property "Reference" "#PWR015" (at 74.93 69.85 0)
       (effects (font (size 1.27 1.27)) hide)
     )
-    (property "Value" "GNDA" (at 68.199 66.7512 90)
+    (property "Value" "GNDA" (at 77.47 67.31 0)
       (effects (font (size 1.27 1.27)) (justify right))
     )
-    (property "Footprint" "" (at 68.072 63.5 0)
+    (property "Footprint" "" (at 74.93 63.5 0)
       (effects (font (size 1.27 1.27)))
     )
-    (property "Datasheet" "" (at 68.072 63.5 0)
+    (property "Datasheet" "" (at 74.93 63.5 0)
       (effects (font (size 1.27 1.27)))
     )
@@
       (effects (font (size 1.27 1.27)) hide)
     )
-    (property "Value" "GNDA" (at 28.067 66.7512 90)
+    (property "Value" "GNDA" (at 30.48 67.31 0)
       (effects (font (size 1.27 1.27)) (justify right))
     )
@@
     )
   )
-  (symbol (lib_id "device:C") (at 68.072 59.69 180) (unit 1)
+  (symbol (lib_id "device:C") (at 74.93 59.69 180) (unit 1)
     (in_bom yes) (on_board yes) (dnp no)
-    (property "Reference" "C7" (at 67.437 62.23 0)
+    (property "Reference" "C7" (at 73.66 57.15 0)
       (effects (font (size 1.27 1.27)) (justify left))
     )
-    (property "Value" "10nF" (at 67.437 57.15 0)
+    (property "Value" "10nF" (at 74.93 62.23 0)
       (effects (font (size 1.27 1.27)) (justify left))
     )
-    (property "Footprint" "Capacitor_SMD:C_0603_1608Metric" (at 67.1068 55.88 0)
+    (property "Footprint" "Capacitor_SMD:C_0603_1608Metric" (at 73.9648 55.88 0)
       (effects (font (size 1.27 1.27)) hide)
     )
-    (property "Datasheet" "" (at 68.072 59.69 0)
+    (property "Datasheet" "" (at 74.93 59.69 0)
       (effects (font (size 1.27 1.27)))
     )
@@
   (symbol (lib_id "device:C") (at 113.03 38.1 0) (unit 1)
     (in_bom yes) (on_board yes) (dnp no)
-    (property "Reference" "C4" (at 113.665 35.56 0)
+    (property "Reference" "C4" (at 109.22 35.56 0)
       (effects (font (size 1.27 1.27)) (justify left))
     )
@@
       (effects (font (size 1.27 1.27)) hide)
     )
-    (property "Value" "GNDA" (at 113.157 45.1612 90)
+    (property "Value" "GNDA" (at 115.57 45.72 0)
       (effects (font (size 1.27 1.27)) (justify right))
     )
@@
   (symbol (lib_id "Device:C") (at 96.52 38.1 0) (unit 1)
     (in_bom yes) (on_board yes) (dnp no)
-    (property "Reference" "C3" (at 96.52 35.56 0)
+    (property "Reference" "C3" (at 92.71 35.56 0)
       (effects (font (size 1.27 1.27)) (justify left))
     )
@@
       (effects (font (size 1.27 1.27)) hide)
     )
-    (property "Value" "GNDA" (at 81.407 66.7512 90)
+    (property "Value" "GNDA" (at 83.82 67.31 0)
       (effects (font (size 1.27 1.27)) (justify right))
     )
@@
       (effects (font (size 1.27 1.27)) hide)
     )
-    (property "Value" "GNDA" (at 96.647 45.1612 90)
+    (property "Value" "GNDA" (at 99.06 45.72 0)
       (effects (font (size 1.27 1.27)) (justify right))
     )
@@
   (symbol (lib_id "Device:C") (at 81.28 59.69 0) (unit 1)
     (in_bom yes) (on_board yes) (dnp no)
-    (property "Reference" "C2" (at 81.28 57.15 0)
+    (property "Reference" "C2" (at 77.47 57.15 0)
       (effects (font (size 1.27 1.27)) (justify left))
     )
